Commit message: Latest code on raspberry pi supporting: - px4-control bench test (in offboard-control-TEST) - safeguards on PX4Control - attempt to scale to PWM (needs to be updated)

File: src/offboardController/assets/x500.urdf (robot description, URDF)
Before this commit: robot x500, 6 links, 5 joints
Links:
- link base_link: mass 1.2105 -> 1.8
